Commit message: updated right wheel in URDF

File: src/sucky_bringup/urdf/robot_core.xacro (robot description, xacro)
@@ -83,6 +83,6 @@
       <parent link="base_link"/>
       <child link="right_wheel"/>
-      <origin xyz="0 ${-wheel_offset_y} 0" rpy="0 0 ${pi}" />
-      <axis xyz="0 -1 0"/>
+      <origin xyz="0 ${-wheel_offset_y} 0" rpy="0 0 0" />
+      <axis xyz="0 1 0"/>
   </joint>
   <link name="right_wheel">
